File: kicad/alcene-board-v1-connectivity-verified.kicad_pcb (KiCad board)
At the start: 2 copper layers, 111.4 x 87.4 mm, 14 parts, among them J1 ESP32-S3-DevKitC-1_J1, J2 USB-C Input, J3 ESP32-S3-DevKitC-1_J3, J4 ILI9341_TFT_14pin, J5 Male Pin Header 1x18 - J1 Sig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, J6 Male Pin Header 1x18 - J3 Sig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, J7 Male Pin Header 2x4 - GND, J8 Male Pin Header 2x4 - 3V3, J9 Male Pin Header 2x4 - VIN 5V, SW1 ESP32-S3 Reset (NO momentary)

Commit message: chore: clean up
Other:
- board size 111.4 x 87.4 mm -> 110 x 88 mm
Changed lines of the file:
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@@
 	)
 	(gr_line
-		(start 33.735715 31.68475)
-		(end 145.089999 31.68475)
+		(start 33.735715 31.0762)
+		(end 143.735715 31.0762)
 		(stroke
-			(width 0.1)
+			(width 0)
 			(type default)
 		)
@@
 	)
 	(gr_line
-		(start 33.735715 119.076198)
-		(end 33.735715 31.68475)
+		(start 33.735715 119.0762)
+		(end 33.735715 31.0762)
 		(stroke
-			(width 0.1)
+			(width 0)
 			(type default)
 		)
@@
 	)
 	(gr_line
-		(start 145.089999 31.68475)
-		(end 145.089999 119.076198)
+		(start 143.735715 31.0762)
+		(end 143.735715 119.0762)
 		(stroke
-			(width 0.1)
+			(width 0)
 			(type default)
 		)
@@
 	)
 	(gr_line
-		(start 145.089999 119.076198)
-		(end 33.735715 119.076198)
+		(start 143.735715 119.0762)
+		(end 33.735715 119.0762)
 		(stroke
-			(width 0.1)
+			(width 0)
 			(type default)
 		)

Commit message: board: fix J1 and J3 spacing to match ESP32 S3 perfectly
Parts:
- moved J3 0.10 mm to (82.4, 48.5)
Routing:
- net GPIO11: track 92.2 -> 188.1 mm, vias 0 -> 1
- net VIN: track 149.5 -> 135.8 mm
- net GPIO8: track 103.1 -> 116.1 mm, vias 0 -> 1
- net GPIO19: track 74.3 -> 62.0 mm
- net RST: track 66.9 -> 72.4 mm, vias 1 -> 3
- net 3V3: track 138.1 -> 142.5 mm, vias 0 -> 1
- net RX: track 39.1 -> 42.4 mm
- net GPIO10: track 103.0 -> 101.4 mm
- net GPIO1: track 39.1 -> 40.6 mm
- net GPIO9: track 97.4 -> 96.1 mm, vias 0 -> 1
- net TX: track 38.0 -> 39.0 mm
- net GPIO15: track 80.8 -> 81.6 mm
- net Net-(J2-PadA5): track 30.8 -> 31.5 mm
- net Net-(J2-PadB5): track 36.7 -> 36.0 mm

Commit message: chore: commit all local changes
Parts:
- moved J4 5.94 mm to (128.6, 113.2)
Routing:
- net GPIO11: track 188.1 -> 93.3 mm, vias 1 -> 0
- net GPIO8: track 116.1 -> 98.8 mm, vias 1 -> 0
- net GPIO19: track 62.0 -> 70.3 mm
- net GPIO12: track 90.2 -> 84.6 mm, vias 0 -> 1
- net GPIO14: track 89.3 -> 84.0 mm
- net GPIO13: track 98.8 -> 94.1 mm
- net GPIO9: track 96.1 -> 91.6 mm, vias 1 -> 0
- net GPIO10: track 101.4 -> 97.2 mm
- net GPIO15: track 81.6 -> 78.8 mm
- net RST: track 72.4 -> 69.7 mm, vias 3 -> 1
- net 3V3: track 142.5 -> 140.2 mm
- net VIN: track 135.8 -> 134.0 mm
Other:
- board size 110 x 88 mm -> 105.5 x 87.4 mm

Commit message: chore: commit all local changes
Parts:
- moved J4 0.12 mm to (128.4, 113.2)
Routing:
- net VIN: track 134.0 -> 145.1 mm, vias 1 -> 0
- net GPIO13: track 94.1 -> 85.2 mm
- net RST: track 69.7 -> 65.6 mm
- net 3V3: track 140.2 -> 136.3 mm, vias 1 -> 0
- net RX: track 42.4 -> 39.0 mm
- net GPIO1: track 40.6 -> 39.0 mm
- net TX: track 39.0 -> 37.9 mm
- net GPIO12: track 84.6 -> 85.6 mm
- net Net-(J2-PadA5): track 31.5 -> 30.8 mm
Other:
- board size 105.5 x 87.4 mm -> 107 x 87 mm
