File: kicad/alcene-board-v1-connectivity-verified.kicad_pcb (KiCad board)
At the start: 2 copper layers, 107 x 87 mm, 14 parts, among them J1 ESP32-S3-DevKitC-1_J1, J2 USB-C Input, J3 ESP32-S3-DevKitC-1_J3, J4 ILI9341_TFT_14pin, J5 Male Pin Header 1x18 - J1 Sig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, J6 Male Pin Header 1x18 - J3 Sig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, J7 Male Pin Header 2x4 - GND, J8 Male Pin Header 2x4 - 3V3, J9 Male Pin Header 2x4 - VIN 5V, SW1 ESP32-S3 Reset (NO momentary)

Commit message: Preserve baseline PCB before alternative layout
Parts:
- added MH1: MountingHole_3mm, MountingHole:MountingHole_3mm, F.Cu at (88.9, 38.8)
- added MH2: MountingHole_3mm, MountingHole:MountingHole_3mm, F.Cu at (134.1, 38.8)
Other:
- board text added: "TFT FAR-END SUPPORT: STANDOFF HEIGHT = J4 HEIGHT + 2.000 MM"
Changed lines of the file:
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@@
 		)
+	)
+	(footprint "MountingHole:MountingHole_3mm"
+		(layer "F.Cu")
+		(at 134.135715 38.75)
+		(property "Reference" "MH2"
+			(at 0 0 0)
+			(layer "F.SilkS")
+			(effects
+				(font
+					(size 1.27 1.27)
+				)
+			)
+		)
+		(property "Value" "MountingHole_3mm"
+			(at 0 0 0)
+			(layer "F.Fab")
+			(effects
+				(font
+					(size 1.27 1.27)
+				)
+			)
+		)
+		(property "Datasheet" ""
+			(at 0 0 0)
+			(layer "F.Fab")
+			(hide yes)
+			(effects
+				(font
+					(size 1.27 1.27)
+				)
+			)
+		)
+		(property "Description" ""
+			(at 0 0 0)
+			(layer "F.Fab")
+			(hide yes)
+			(effects
+				(font
+					(size 1.27 1.27)
+				)
+			)
+		)
+		(duplicate_pad_numbers_are_jumpers no)
+		(pad "" np_thru_hole circle
+			(at 0 0)
+			(size 3 3)
+			(drill 3)
+			(layers "*.Mask")
+		)
+		(embedded_fonts no)
 	)
 	(footprint "Connector_PinSocket_2.54mm:PinSocket_1x22_P2.54mm_Vertical"
@@
 		)
 	)
+	(footprint "MountingHole:MountingHole_3mm"
+		(layer "F.Cu")
+		(at 88.935715 38.75)
+		(property "Reference" "MH1"
+			(at 0 0 0)
+			(layer "F.SilkS")
+			(effects
+				(font
+					(size 1.27 1.27)
+				)
+			)
+		)
+		(property "Value" "MountingHole_3mm"
+			(at 0 0 0)
+			(layer "F.Fab")
+			(effects
+				(font
+					(size 1.27 1.27)
+				)
+			)
+		)
+		(property "Datasheet" ""
+			(at 0 0 0)
+			(layer "F.Fab")
+			(hide yes)
+			(effects
+				(font
+					(size 1.27 1.27)
+				)
+			)
+		)
+		(property "Description" ""
+			(at 0 0 0)
+			(layer "F.Fab")
+			(hide yes)
+			(effects
+				(font
+					(size 1.27 1.27)
+				)
+			)
+		)
+		(duplicate_pad_numbers_are_jumpers no)
+		(pad "" np_thru_hole circle
+			(at 0 0)
+			(size 3 3)
+			(drill 3)
+			(layers "*.Mask")
+		)
+		(embedded_fonts no)
+	)
 	(footprint "Capacitor_SMD:C_0805_2012Metric"
 		(layer "F.Cu")
@@
 		(layer "F.SilkS")
 		(effects
+			(font
+				(size 1 1)
+				(thickness 0.15)
+			)
+		)
+	)
+	(gr_text "TFT FAR-END SUPPORT: STANDOFF HEIGHT = J4 HEIGHT + 2.000 MM"
+		(at 95 32 0)
+		(layer "F.SilkS")
+		(effects

Commit message: board: RC 3.1 - standoff
Other:
- board text removed: "TFT FAR-END SUPPORT: STANDOFF HEIGHT = J4 HEIGHT + 2.000 MM"
Changed lines of the file:
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@@
 		(at 134.135715 38.75)
 		(property "Reference" "MH2"
-			(at 0 0 0)
+			(at 0.014285 2.85 0)
 			(layer "F.SilkS")
 			(effects
@@
 		(at 88.935715 38.75)
 		(property "Reference" "MH1"
-			(at 0 0 0)
+			(at 0 2.85 0)
 			(layer "F.SilkS")
 			(effects
@@
 		(layer "F.SilkS")
 		(effects
-			(font
-				(size 1 1)
-				(thickness 0.15)
-			)
-		)
-	)
-	(gr_text "TFT FAR-END SUPPORT: STANDOFF HEIGHT = J4 HEIGHT + 2.000 MM"
-		(at 95 32 0)
-		(layer "F.SilkS")
-		(effects
