File: kicad/alcene-board-v1.kicad_pcb (KiCad board)
At the start: 2 copper layers, 107 x 87 mm, 16 parts, among them J1 ESP32-S3-DevKitC-1_J1, J2 USB-C Input, J3 ESP32-S3-DevKitC-1_J3, J4 ILI9341_TFT_14pin, J5 Male Pin Header 1x18 - J1 Sig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, J6 Male Pin Header 1x18 - J3 Sig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, J7 Male Pin Header 2x4 - GND, J8 Male Pin Header 2x4 - 3V3, J9 Male Pin Header 2x4 - VIN 5V, SW1 ESP32-S3 Reset (NO momentary)

Commit message: cp: Rotate J4 connector 180 degrees and reroute affected nets
Parts:
- moved J4 33.0 mm to (95.4, 113.2), turned to 90 degrees
Routing:
- net GND: track 27.5 -> 191.3 mm
- net GPIO11: track 93.2 -> 228.8 mm
- net GPIO13: track 85.2 -> 216.5 mm
- net GPIO12: track 85.6 -> 190.4 mm, vias 1 -> 0
- net 3V3: track 136.3 -> 201.0 mm
- net GPIO9: track 91.5 -> 58.0 mm
- net GPIO8: track 98.7 -> 67.8 mm
- net RST: track 65.6 -> 35.2 mm
- net GPIO10: track 97.0 -> 114.5 mm
- net GPIO14: track 83.9 -> 98.6 mm
- net VIN: track 145.3 -> 130.6 mm
- net GPIO38: track 39.0 -> 33.6 mm
- net GPIO45: track 39.0 -> 33.6 mm
- net GPIO15: track 78.4 -> 76.0 mm

Commit message: cp: 2
Routing:
- net GND: track 191.3 -> 28.1 mm
- net GPIO11: track 228.8 -> 97.6 mm, vias 0 -> 1
- net GPIO13: track 216.5 -> 95.8 mm
- net GPIO12: track 190.4 -> 96.1 mm, vias 0 -> 1
- net RST: track 35.2 -> 90.9 mm, vias 1 -> 2
- net GPIO15: track 76.0 -> 124.2 mm, vias 0 -> 1
- net 3V3: track 201.0 -> 157.5 mm, vias 0 -> 1
- net GPIO9: track 58.0 -> 77.5 mm
- net GPIO10: track 114.5 -> 104.8 mm, vias 0 -> 1
- net GPIO8: track 67.8 -> 76.6 mm
- net GPIO14: track 98.6 -> 90.3 mm
- net GPIO38: track 33.6 -> 38.9 mm
- net GPIO45: track 33.6 -> 38.9 mm
- net VIN: track 130.6 -> 131.5 mm
