File: kicad/ALCENE_TFT_ROUTING_VERIFIED_RELEASE_20261024.kicad_pcb (KiCad board)
At the start: 2 copper layers, 107 x 87 mm, 16 parts, among them J1 ESP32-S3-DevKitC-1_J1, J2 USB-C Input, J3 ESP32-S3-DevKitC-1_J3, J4 ILI9341_TFT_14pin, J5 Male Pin Header 1x18 - J1 Sig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, J6 Male Pin Header 1x18 - J3 Sig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, J7 Male Pin Header 2x4 - GND, J8 Male Pin Header 2x4 - 3V3, J9 Male Pin Header 2x4 - VIN 5V, SW1 ESP32-S3 Reset (NO momentary)

Commit message: cp: 3
Routing:
- net VIN: track 131.5 -> 152.3 mm
- net GND: track 28.1 -> 41.1 mm
- net RST: track 90.9 -> 94.9 mm, vias 2 -> 1
Other:
- board text added: "5V"
- board text removed: "VIN"
