File: kicad/ALCENE_PRODUCTION_QC_FIXED_20261024.kicad_pcb (KiCad board)
At the start: 2 copper layers, 107 x 87 mm, 16 parts, among them J1 ESP32-S3-DevKitC-1_J1, J2 USB-C Input, J3 ESP32-S3-DevKitC-1_J3, J4 ILI9341_TFT_14pin, J5 Male Pin Header 1x18 - J1 Sig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, J6 Male Pin Header 1x18 - J3 Sig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, J7 Male Pin Header 2x4 - GND, J8 Male Pin Header 2x4 - 3V3, J9 Male Pin Header 2x4 - VIN 5V, SW1 ESP32-S3 Reset (NO momentary)

Commit message: chore: commit all local changes
Routing:
- net RST: track 0.00 -> 90.9 mm, vias 0 -> 2
Changed lines of the file:
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@@
+	)
+	(segment
+		(start 82.7767 100.57)
+		(end 83.6 99.7467)
+		(width 0.2)
+		(layer "F.Cu")
+		(net "RST")
+	)
+	(segment
+		(start 57 111.3)
+		(end 57 110.377)
+		(width 0.2)
+		(layer "F.Cu")
+		(net "RST")
+	)
+	(segment
+		(start 78.932 94.9834)
+		(end 77.4167 94.9834)
+		(width 0.2)
+		(layer "F.Cu")
+		(net "RST")
+	)
+	(segment
+		(start 66.8071 100.57)
+		(end 82.7767 100.57)
+		(width 0.2)
+		(layer "F.Cu")
+		(net "RST")
+	)
+	(segment
+		(start 82.0066 98.058)
+		(end 78.932 94.9834)
+		(width 0.2)
+		(layer "F.Cu")
+		(net "RST")
+	)
+	(segment
+		(start 82.0984 98.1498)
+		(end 82.0066 98.058)
+		(width 0.2)
+		(layer "F.Cu")
+		(net "RST")
+	)
+	(segment
+		(start 83.6 98.1498)
+		(end 82.0984 98.1498)
+		(width 0.2)
+		(layer "F.Cu")
+		(net "RST")
+	)
+	(segment
+		(start 83.6 99.7467)
+		(end 83.6 98.1498)
+		(width 0.2)
+		(layer "F.Cu")
+		(net "RST")
+	)
+	(segment
+		(start 57 110.377)
+		(end 66.8071 100.57)
+		(width 0.2)
+		(layer "F.Cu")
+		(net "RST")
+	)
+	(via
+		(at 77.4167 94.9834)
+		(size 0.6)
+		(drill 0.3)
+		(layers "F.Cu" "B.Cu")
+		(net "RST")
+	)
+	(via
+		(at 57 110.377)
+		(size 0.6)
+		(drill 0.3)
+		(layers "F.Cu" "B.Cu")
+		(net "RST")
+	)
+	(segment
+		(start 77.4167 94.9834)
+		(end 58.9939 76.5606)
+		(width 0.2)
+		(layer "B.Cu")
+		(net "RST")
+	)
+	(segment
+		(start 58.9939 76.5606)
+		(end 58.9939 55.5739)
+		(width 0.2)
+		(layer "B.Cu")
+		(net "RST")
+	)
+	(segment
+		(start 58.9939 55.5739)
+		(end 57 53.58)
+		(width 0.2)
+		(layer "B.Cu")
+		(net "RST")
 	)
 	(segment
