File: kicad/alcene-board-v2-rebased-zero-drc.kicad_pcb (KiCad board)
At the start: 2 copper layers, 109.3 x 87.1 mm, 16 parts, among them J1 ESP32-S3-DevKitC-1_J1, J2 USB-C Input, J3 ESP32-S3-DevKitC-1_J3, J4 ILI9341_TFT_14pin, J5 Male Pin Header 1x18 - J1 Sig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, J6 Male Pin Header 1x18 - J3 Sig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, J7 Male Pin Header 2x4 - GND, J8 Male Pin Header 2x4 - 3V3, J9 Male Pin Header 2x4 - VIN 5V, SW1 ESP32-S3 Reset (NO momentary)

Commit message: feat: final layout
Routing:
- net GND: track 253.5 -> 246.4 mm
- net GPIO12: track 91.6 -> 87.4 mm
- net 3V3: track 140.5 -> 137.4 mm
- net GPIO11: track 102.3 -> 99.2 mm
- net GPIO13: track 81.1 -> 83.6 mm, vias 4 -> 2
- net GPIO15: track 100.8 -> 99.3 mm
- net GPIO10: track 103.2 -> 101.7 mm
- net GPIO9: track 94.7 -> 93.1 mm
- net GPIO8: track 100.4 -> 98.8 mm
- net GPIO14: track 74.4 -> 75.4 mm, vias 1 -> 0
Changed lines of the file:
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@@
-	)
-	(segment
-		(start 76.6 112.5)
-		(end 76.6 115.44)
-		(width 0.2)
-		(layer "F.Cu")
-		(net "GND")
 	)
 	(segment
 		(start 143.295 111.84)
 		(end 142 111.84)
-		(width 0.2)
-		(layer "F.Cu")
-		(net "GND")
-	)
-	(segment
-		(start 74 112.5)
-		(end 76.6 112.5)
 		(width 0.2)
 		(layer "F.Cu")
@@
 	)
 	(segment
+		(start 87.1051 115.118)
+		(end 98.524 115.118)
+		(width 0.2)
+		(layer "F.Cu")
+		(net "GND")
+	)
+	(segment
 		(start 129.56 103.34)
 		(end 122.824 103.34)
@@
 	)
 	(segment
-		(start 60.75 113.25)
-		(end 60.75 118.85)
-		(width 0.2)
-		(layer "F.Cu")
-		(net "GND")
-	)
-	(segment
 		(start 141.49 103.34)
 		(end 144.6 103.34)
@@
 	)
 	(segment
-		(start 87.1051 115.118)
-		(end 98.524 115.118)
-		(width 0.2)
-		(layer "F.Cu")
-		(net "GND")
-	)
-	(segment
 		(start 121.58 102.613)
 		(end 104.887 102.613)
@@
 		(start 104.16 109.482)
 		(end 112.869 118.191)
+		(width 0.2)
+		(layer "F.Cu")
+		(net "GND")
+	)
+	(segment
+		(start 60.75 113.25)
+		(end 60.75 117.3)
 		(width 0.2)
 		(layer "F.Cu")
@@
 	(segment
 		(start 58.21 113.25)
-		(end 58.21 118.85)
+		(end 58.21 117.3)
 		(width 0.2)
 		(layer "F.Cu")
@@
 	)
 	(segment
+		(start 75.99 113.25)
+		(end 75.99 117.3)
+		(width 0.2)
+		(layer "B.Cu")
+		(net "3V3")
+	)
+	(segment
 		(start 102.92 53.7799)
 		(end 104.16 52.54)
@@
 		(start 105.31 89.37)
 		(end 105.31 77.7878)
-		(width 0.2)
-		(layer "B.Cu")
-		(net "3V3")
-	)
-	(segment
-		(start 75.99 113.25)
-		(end 75.99 118.85)
 		(width 0.2)
 		(layer "B.Cu")
@@
 	(segment
 		(start 63.29 113.25)
-		(end 63.29 118.85)
+		(end 63.29 117.3)
 		(width 0.2)
 		(layer "B.Cu")
@@
 	(segment
 		(start 65.83 113.25)
-		(end 65.83 118.85)
+		(end 65.83 117.3)
 		(width 0.2)
 		(layer "B.Cu")
@@
 	(segment
 		(start 68.37 113.25)
-		(end 68.37 118.85)
+		(end 68.37 117.3)
 		(width 0.2)
 		(layer "B.Cu")
@@
 	)
 	(segment
-		(start 70.91 113.25)
-		(end 70.91 118.85)
+		(start 86.15 113.25)
+		(end 86.15 117.3)
 		(width 0.2)
 		(layer "B.Cu")
@@
 	)
 	(segment
-		(start 86.15 113.25)
-		(end 86.15 118.85)
-		(width 0.2)
-		(layer "B.Cu")
-		(net "GPIO11")
-	)
-	(segment
 		(start 105.15 92.543)
 		(end 105.15 91.6296)
@@
 	)
 	(segment
+		(start 70.91 113.25)
+		(end 70.91 117.3)
+		(width 0.2)
+		(layer "B.Cu")
+		(net "GPIO11")
+	)
+	(segment
+		(start 73.45 117.3)
+		(end 73.45 118.55)
+		(width 0.2)
+		(layer "F.Cu")
+		(net "GPIO12")
+	)
+	(segment
+		(start 81.07 118.55)
+		(end 81.07 117.3)
+		(width 0.2)
+		(layer "F.Cu")
+		(net "GPIO12")
+	)
+	(segment
 		(start 143.199 91.9844)
 		(end 144.314 93.1)
@@
 	)
 	(segment
+		(start 73.45 118.55)
+		(end 81.07 118.55)
+		(width 0.2)
+		(layer "F.Cu")
+		(net "GPIO12")
+	)
+	(segment
 		(start 104.16 93.18)
 		(end 105.356 91.9844)
@@
 	)
 	(segment
-		(start 79.9091 114.411)
-		(end 81.07 113.25)
-		(width 0.2)
-		(layer "B.Cu")
-		(net "GPIO12")
-	)
-	(segment
-		(start 74.6109 114.411)
-		(end 75.29 114.411)
-		(width 0.2)
-		(layer "B.Cu")
-		(net "GPIO12")
-	)
-	(segment
-		(start 73.45 113.25)
-		(end 74.6109 114.411)
-		(width 0.2)
-		(layer "B.Cu")
-		(net "GPIO12")
-	)
-	(segment
-		(start 76.69 114.411)
-		(end 79.9091 114.411)
-		(width 0.2)
-		(layer "B.Cu")
-		(net "GPIO12")
-	)
-	(segment
-		(start 81.07 113.25)
-		(end 81.07 118.85)
-		(width 0.2)
-		(layer "B.Cu")
-		(net "GPIO12")
-	)
-	(segment
 		(start 81.07 113.25)
 		(end 101.14 93.18)
@@
 	)
 	(segment
-		(start 73.45 113.25)
-		(end 73.45 118.85)
+		(start 81.07 113.25)
+		(end 81.07 117.3)
 		(width 0.2)
 		(layer "B.Cu")
@@
 	)
 	(segment
+		(start 132.416 94.4091)
+		(end 133.246 94.4091)
+		(width 0.2)
+		(layer "F.Cu")
+		(net "GPIO13")
+	)
+	(segment
+		(start 132.255 94.5698)
+		(end 132.416 94.4091)
+		(width 0.2)
+		(layer "F.Cu")
+		(net "GPIO13")
+	)
+	(segment
+		(start 104.16 95.72)
+		(end 122.052 95.72)
+		(width 0.2)
+		(layer "F.Cu")
+		(net "GPIO13")
+	)
+	(segment
 		(start 78.53 116)
 		(end 88.69 116)
-		(width 0.2)
-		(layer "F.Cu")
-		(net "GPIO13")
-	)
-	(segment
-		(start 132.416 94.4091)
-		(end 133.246 94.4091)
-		(width 0.2)
-		(layer "F.Cu")
-		(net "GPIO13")
-	)
-	(segment
-		(start 132.255 94.5698)
-		(end 132.416 94.4091)
-		(width 0.2)
-		(layer "F.Cu")
-		(net "GPIO13")
-	)
-	(segment
-		(start 104.16 95.72)
-		(end 122.052 95.72)
 		(width 0.2)
 		(layer "F.Cu")
@@
 		(net "GPIO13")
 	)
-	(via
-		(at 78.53 116)
-		(size 0.6)
-		(drill 0.3)
-		(layers "F.Cu" "B.Cu")
-		(net "GPIO13")
-	)
-	(via
-		(at 88.69 116)
-		(size 0.6)
-		(drill 0.3)
-		(layers "F.Cu" "B.Cu")
-		(net "GPIO13")
-	)
 	(segment
 		(start 105.35 98.8118)
@@
 	)
 	(segment
+		(start 88.69 113.25)
+		(end 88.69 117.3)
+		(width 0.2)
+		(layer "B.Cu")
+		(net "GPIO13")
+	)
+	(segment
 		(start 104.632 99.53)
 		(end 102.41 99.53)
@@
 	(segment
 		(start 78.53 116)
-		(end 78.53 118.85)
+		(end 78.53 117.3)
 		(width 0.2)
 		(layer "B.Cu")
@@
 	)
 	(segment
-		(start 83.61 115.8)
-		(end 83.61 118.85)
-		(width 0.2)
-		(layer "F.Cu")
-		(net "GPIO14")
-	)
-	(segment
 		(start 143.729 99.4506)
 		(end 145 98.18)
@@
 	)
 	(segment
-		(start 83.61 115.8)
-		(end 87.42 115.8)
-		(width 0.2)
-		(layer "F.Cu")
-		(net "GPIO14")
-	)
-	(via
-		(at 87.42 115.8)
-		(size 0.6)
-		(drill 0.3)
-		(layers "F.Cu" "B.Cu")
-		(net "GPIO14")
-	)
-	(segment
 		(start 104.16 98.26)
 		(end 102.026 98.26)
@@
 	)
 	(segment
+		(start 87.42 112.866)
+		(end 87.42 118.55)
+		(width 0.2)
+		(layer "B.Cu")
+		(net "GPIO14")
+	)
+	(segment
+		(start 87.42 118.55)
+		(end 83.61 118.55)
+		(width 0.2)
+		(layer "B.Cu")
+		(net "GPIO14")
+	)
+	(segment
+		(start 83.61 118.55)
+		(end 83.61 117.3)
+		(width 0.2)
+		(layer "B.Cu")
+		(net "GPIO14")
+	)
+	(segment
 		(start 102.026 98.26)
 		(end 87.42 112.866)
@@
 	)
 	(segment
-		(start 87.42 115.8)
-		(end 87.42 112.866)
-		(width 0.2)
-		(layer "B.Cu")
-		(net "GPIO14")
-	)
-	(segment
 		(start 143.199 66.5844)
 		(end 144.314 67.7)
@@
 	(segment
 		(start 91.23 113.25)
-		(end 91.23 118.85)
-		(width 0.2)
-		(layer "B.Cu")
+		(end 91.23 117.3)
+		(width 0.2)
+		(layer "B.Cu")

Commit message: feat: best practice wiring
Routing:
- net GND: track 246.4 -> 240.2 mm
- net 3V3: track 137.4 -> 131.8 mm
- net GPIO10: track 101.7 -> 96.7 mm
- net VIN: track 170.2 -> 167.5 mm
- net GPIO11: track 99.2 -> 97.7 mm
- net Net-(J2-PadB5): track 10.9 -> 10.2 mm
- net GPIO12: track 87.4 -> 86.8 mm
Other:
- board text removed: "2.8 INCH TFT DISPLAY AREA 50.0 x 85.0 mm (Dwg reservation)"
